Commit message: docker simulation

File: src/abb_irb120_description/urdf/irb120_3_60_macro.xacro (robot description, xacro)
@@ -142,6 +142,6 @@
       <parent link="${prefix}base_link"/>
       <child link="${prefix}link_1"/>
-      <limit effort="0" lower="${radians(-165)}" upper="${radians(165)}" velocity="${radians(250)}"/>
-      <dynamics damping="0.0" friction="0.0"/>
+      <limit effort="200" lower="${radians(-165)}" upper="${radians(165)}" velocity="${radians(250)}"/>
+      <dynamics damping="5.0" friction="0.2"/>
     </joint>
     <joint type="revolute" name="${prefix}joint_2">
@@ -150,6 +150,6 @@
       <parent link="${prefix}link_1"/>
       <child link="${prefix}link_2"/>
-      <limit effort="0" lower="${radians(-110)}" upper="${radians(110)}" velocity="${radians(250)}"/>
-      <dynamics damping="0.0" friction="0.0"/>
+      <limit effort="200" lower="${radians(-110)}" upper="${radians(110)}" velocity="${radians(250)}"/>
+      <dynamics damping="5.0" friction="0.2"/>
     </joint>
     <joint type="revolute" name="${prefix}joint_3">
@@ -158,6 +158,6 @@
       <parent link="${prefix}link_2"/>
       <child link="${prefix}link_3"/>
-      <limit effort="0" lower="${radians(-110)}" upper="${radians(70)}" velocity="${radians(250)}"/>
-      <dynamics damping="0.0" friction="0.0"/>
+      <limit effort="200" lower="${radians(-110)}" upper="${radians(70)}" velocity="${radians(250)}"/>
+      <dynamics damping="5.0" friction="0.2"/>
     </joint>
     <joint type="revolute" name="${prefix}joint_4">
@@ -166,6 +166,6 @@
       <parent link="${prefix}link_3"/>
       <child link="${prefix}link_4"/>
-      <limit effort="0" lower="${radians(-160)}" upper="${radians(160)}" velocity="${radians(320)}"/>
-      <dynamics damping="0.0" friction="0.0"/>
+      <limit effort="200" lower="${radians(-160)}" upper="${radians(160)}" velocity="${radians(320)}"/>
+      <dynamics damping="5.0" friction="0.2"/>
     </joint>
     <joint type="revolute" name="${prefix}joint_5">
@@ -174,6 +174,6 @@
       <parent link="${prefix}link_4"/>
       <child link="${prefix}link_5"/>
-      <limit effort="0" lower="${radians(-120)}" upper="${radians(120)}" velocity="${radians(320)}"/>
-      <dynamics damping="0.0" friction="0.0"/>
+      <limit effort="200" lower="${radians(-120)}" upper="${radians(120)}" velocity="${radians(320)}"/>
+      <dynamics damping="5.0" friction="0.2"/>
     </joint>
     <joint type="revolute" name="${prefix}joint_6">
@@ -182,6 +182,6 @@
       <parent link="${prefix}link_5"/>
       <child link="${prefix}link_6"/>
-      <limit effort="0" lower="${radians(-400)}" upper="${radians(400)}" velocity="${radians(420)}"/>
-      <dynamics damping="0.0" friction="0.0"/>
+      <limit effort="200" lower="${radians(-400)}" upper="${radians(400)}" velocity="${radians(420)}"/>
+      <dynamics damping="5.0" friction="0.2"/>
     </joint>
     <!-- end of joint list -->

File: src/abb_irb120_moveit/config/abb_irb120_3_60.ros2_control.xacro (robot description, xacro)
@@ -3,8 +3,7 @@
     <xacro:macro name="abb_irb120_3_60_ros2_control" params="name initial_positions_file">
         <xacro:property name="initial_positions" value="${xacro.load_yaml(initial_positions_file)['initial_positions']}"/>
-        <ros2_control name="${name}" type="system">
+        <ros2_control name="GazeboSimSystem" type="system">
             <hardware>
-                <!-- By default, set up controllers for simulation. This won't work on real hardware -->
-                <plugin>mock_components/GenericSystem</plugin>
+                <plugin>gz_ros2_control/GazeboSimSystem</plugin>
             </hardware>
             <joint name="joint_1">
@@ -51,4 +50,9 @@
             </joint>
         </ros2_control>
+        <gazebo>
+            <plugin filename="libgz_ros2_control-system.so" name="gz_ros2_control::GazeboSimROS2ControlPlugin">
+                <parameters>$(find abb_irb120_moveit)/config/ros2_controllers.yaml</parameters>
+            </plugin>
+        </gazebo>
     </xacro:macro>
 </robot>

File: src/abb_irb120_moveit/config/abb_irb120_3_60.urdf.xacro (robot description, xacro)
@@ -3,7 +3,13 @@
     <xacro:arg name="initial_positions_file" default="initial_positions.yaml" />
     <!-- Import abb_irb120_3_60 urdf file -->
-    <xacro:include filename="$(find abb_irb120_description)/urdf\irb120_3_60.xacro" />
+    <xacro:include filename="$(find abb_irb120_description)/urdf/irb120_3_60.xacro" />
     <!-- Import control_xacro -->
     <xacro:include filename="abb_irb120_3_60.ros2_control.xacro" />
-    <xacro:abb_irb120_3_60_ros2_control name="FakeSystem" initial_positions_file="$(arg initial_positions_file)"/>
+    <link name="world"/>
+    <joint name="world_to_base" type="fixed">
+        <parent link="world"/>
+        <child link="base_link"/>
+        <origin xyz="0 0 0" rpy="0 0 0"/>
+    </joint>
+    <xacro:abb_irb120_3_60_ros2_control name="GazeboSimSystem" initial_positions_file="$(arg initial_positions_file)"/>
 </robot>
