Commit message: gripper mimic fix

File: src/abb_irb120_description/urdf/gripper_macro.xacro (robot description, xacro)
@@ -84,4 +84,5 @@
         <axis xyz="0 -1 0"/>
         <limit lower="0.0" upper="0.01" effort="150" velocity="0.05"/>
+        <dynamics damping="5.0" friction="0.5"/>
     </joint>
     <joint name="${prefix}right_finger_joint" type="prismatic">
@@ -90,5 +91,7 @@
         <origin xyz="0 0 0" rpy="0 0 0"/>
         <axis xyz="0 1 0"/>
+        <mimic joint="${prefix}left_finger_joint" multiplier="1.0" offset="0.0"/>
         <limit lower="0.0" upper="0.01" effort="150" velocity="0.05"/>
+        <dynamics damping="5.0" friction="0.5"/>
     </joint>
     <link name="${prefix}gripper_tcp"/>

File: src/abb_irb120_moveit/config/abb_irb120_3_60.ros2_control.xacro (robot description, xacro)
@@ -57,5 +57,4 @@
             </joint>
             <joint name="right_finger_joint">
-                <command_interface name="position"/>
                 <state_interface name="position">
                 <param name="initial_value">${initial_positions['right_finger_joint']}</param>

Commit message: egm controller execution

File: src/abb_irb120_description/urdf/gripper_macro.xacro (robot description, xacro)
@@ -101,4 +101,10 @@
         <origin xyz="0 0 0.1353" rpy="0 0 0"/>
     </joint>
+    <link name="${prefix}gripper_tcp_calibrated"/>
+    <joint name="${prefix}gripper_base-gripper_tcp_calibrated" type="fixed">
+        <parent link="${prefix}gripper_base"/>
+        <child link="${prefix}gripper_tcp_calibrated"/>
+        <origin xyz="0 0 0.139" rpy="0 0 ${radians(45)}"/>
+    </joint>
   </xacro:macro>
 </robot>

Commit message: Ongoing bug fixing

File: src/abb_irb120_description/urdf/gripper_macro.xacro (robot description, xacro)
@@ -28,7 +28,7 @@
     <link name="${prefix}left_finger">
       <inertial>
-        <mass value="0.1"/>
+        <mass value="0.5"/>
         <origin xyz="0 0 0" rpy="0 0 0"/>
-        <inertia ixx="1e-6" ixy="0" ixz="0" iyy="1e-6" iyz="0" izz="1e-6"/>
+        <inertia ixx="1e-4" ixy="0" ixz="0" iyy="1e-4" iyz="0" izz="1e-4"/>
       </inertial>
       <collision name="collision">
@@ -46,7 +46,7 @@
     <link name="${prefix}right_finger">
       <inertial>
-        <mass value="0.1"/>
+        <mass value="0.5"/>
         <origin xyz="0 0 0" rpy="0 0 0"/>
-        <inertia ixx="1e-6" ixy="0" ixz="0" iyy="1e-6" iyz="0" izz="1e-6"/>
+        <inertia ixx="1e-4" ixy="0" ixz="0" iyy="1e-4" iyz="0" izz="1e-4"/>
       </inertial>
       <collision name="collision">
@@ -63,16 +63,16 @@
     </link>
     <gazebo reference="${prefix}left_finger">
-      <mu1>5.0</mu1>
-      <mu2>5.0</mu2>
-      <kp>10000000.0</kp>
-      <kd>10000.0</kd>
+      <mu1>20.0</mu1>
+      <mu2>20.0</mu2>
+      <kp>1000000000.0</kp>
+      <kd>1000000.0</kd>
       <maxVel>0.01</maxVel>
       <minDepth>0.001</minDepth>
     </gazebo>
     <gazebo reference="${prefix}right_finger">
-      <mu1>5.0</mu1>
-      <mu2>5.0</mu2>
-      <kp>10000000.0</kp>
-      <kd>10000.0</kd>
+      <mu1>20.0</mu1>
+      <mu2>20.0</mu2>
+      <kp>1000000000.0</kp>
+      <kd>1000000.0</kd>
       <maxVel>0.01</maxVel>
       <minDepth>0.001</minDepth>
@@ -83,6 +83,6 @@
         <origin xyz="0 0 0" rpy="0 0 0"/>
         <axis xyz="0 -1 0"/>
-        <limit lower="-0.001" upper="0.011" effort="300" velocity="0.05"/>
-        <dynamics damping="5.0" friction="0.5"/>
+        <limit lower="-0.001" upper="0.025" effort="1000" velocity="0.05"/>
+        <dynamics damping="1.0" friction="0.1"/>
     </joint>
     <joint name="${prefix}right_finger_joint" type="prismatic">
@@ -92,7 +92,15 @@
         <axis xyz="0 1 0"/>
         <mimic joint="${prefix}left_finger_joint" multiplier="1.0" offset="0.0"/>
-        <limit lower="-0.001" upper="0.011" effort="300" velocity="0.05"/>
-        <dynamics damping="5.0" friction="0.5"/>
+        <limit lower="-0.001" upper="0.025" effort="1000" velocity="0.05"/>
+        <dynamics damping="1.0" friction="0.1"/>
     </joint>
+    <gazebo>
+      <plugin filename="gz-sim-mimic-system" name="gz::sim::systems::Mimic">
+        <joint>left_finger_joint</joint>
+        <mimic_joint>right_finger_joint</mimic_joint>
+        <multiplier>1.0</multiplier>
+        <offset>0.0</offset>
+      </plugin>
+    </gazebo>
     <link name="${prefix}gripper_tcp"/>
     <joint name="${prefix}gripper_base-gripper_tcp" type="fixed">

File: src/abb_irb120_moveit/config/abb_irb120_3_60.ros2_control.xacro (robot description, xacro)
@@ -57,4 +57,5 @@
             </joint>
             <joint name="right_finger_joint">
+                <command_interface name="position"/>
                 <state_interface name="position">
                 <param name="initial_value">${initial_positions['right_finger_joint']}</param>

Commit message: bug fixing for trajectory planner.

File: src/abb_irb120_description/urdf/gripper_macro.xacro (robot description, xacro)
@@ -63,6 +63,6 @@
     </link>
     <gazebo reference="${prefix}left_finger">
-      <mu1>20.0</mu1>
-      <mu2>20.0</mu2>
+      <mu1>1000.0</mu1>
+      <mu2>1000.0</mu2>
       <kp>1000000000.0</kp>
       <kd>1000000.0</kd>
@@ -71,6 +71,6 @@
     </gazebo>
     <gazebo reference="${prefix}right_finger">
-      <mu1>20.0</mu1>
-      <mu2>20.0</mu2>
+      <mu1>1000.0</mu1>
+      <mu2>1000.0</mu2>
       <kp>1000000000.0</kp>
       <kd>1000000.0</kd>
@@ -83,5 +83,5 @@
         <origin xyz="0 0 0" rpy="0 0 0"/>
         <axis xyz="0 -1 0"/>
-        <limit lower="-0.001" upper="0.025" effort="1000" velocity="0.05"/>
+        <limit lower="-0.001" upper="0.025" effort="5000" velocity="0.05"/>
         <dynamics damping="1.0" friction="0.1"/>
     </joint>
@@ -92,15 +92,7 @@
         <axis xyz="0 1 0"/>
         <mimic joint="${prefix}left_finger_joint" multiplier="1.0" offset="0.0"/>
-        <limit lower="-0.001" upper="0.025" effort="1000" velocity="0.05"/>
+        <limit lower="-0.001" upper="0.025" effort="5000" velocity="0.05"/>
         <dynamics damping="1.0" friction="0.1"/>
     </joint>
-    <gazebo>
-      <plugin filename="gz-sim-mimic-system" name="gz::sim::systems::Mimic">
-        <joint>left_finger_joint</joint>
-        <mimic_joint>right_finger_joint</mimic_joint>
-        <multiplier>1.0</multiplier>
-        <offset>0.0</offset>
-      </plugin>
-    </gazebo>
     <link name="${prefix}gripper_tcp"/>
     <joint name="${prefix}gripper_base-gripper_tcp" type="fixed">
